Commit message: add RGBD camera

File: hurba_mapping/urdf/hurba_mecanum.xacro (robot description, xacro)
@@ -32,4 +32,9 @@
     <axis xyz="0 1 0" rpy="0 0 0"/>
   </joint>
+  <joint type="fixed" name="camera_optical_joint">
+    <origin xyz="0 0 0" rpy="-1.5707 0 -1.5707"/>
+    <child link="camera_link_optical"/>
+    <parent link="camera_link"/>
+  </joint>
   <joint type="fixed" name="scan_joint">
     <origin xyz="0.0 0 0.38" rpy="0 0 0"/>
@@ -162,4 +167,6 @@
       </geometry>
     </visual>
+  </link>
+  <link name="camera_link_optical">
   </link>
   <!--lidar-->

Commit message: fix a bug that referenced a path outside of this project

File: hurba_mapping/urdf/hurba_mecanum.xacro (robot description, xacro)
@@ -65,5 +65,5 @@
       <geometry>
         <!--box size=".4 .4 .4"/-->
-        <mesh filename = "package://hurba_robot/meshes/chassis.dae"/>
+        <mesh filename = "package://hurba_mapping/meshes/chassis.dae"/>
       </geometry>
     </visual>
@@ -113,5 +113,5 @@
       <origin xyz="0.0 0 0" rpy=" 0 1.5708 1.5708"/>
       <geometry>
-        <mesh filename = "package://hurba_robot/meshes/wheel.dae"/>
+        <mesh filename = "package://hurba_mapping/meshes/wheel.dae"/>
         <!--cylinder radius = ".1" length = ".08"/-->
       </geometry>
@@ -138,5 +138,5 @@
       <origin xyz="0 0 0" rpy=" 0 1.5708 1.5708"/>
       <geometry>
-        <mesh filename = "package://hurba_robot/meshes/wheel.dae"/>
+        <mesh filename = "package://hurba_mapping/meshes/wheel.dae"/>
         <!--cylinder radius = ".1" length = ".08"/-->
       </geometry>
@@ -190,5 +190,5 @@
       <origin xyz="0 0 0" rpy=" 0 0 0"/>
       <geometry>
-        <mesh filename = "package://hurba_robot/meshes/hokuyo.dae"/>
+        <mesh filename = "package://hurba_mapping/meshes/hokuyo.dae"/>
       </geometry>
     </visual>
